File: traffic_light.brd (EAGLE design)
At the start: 100 x 80 mm, 58 parts, among them IC1 74LS48N, IC2 74LS48N, IC3 NE555N, IC4 74LS48N, IC5 74LS48N, IC6 74190N, IC7 74190N

Commit message: commit
Parts:
- removed IC1, IC2, IC4, IC5: 74LS48N, 74xx-eu:DIL16
- removed R1, R10, R11, R12, R13, R14, R15, R16, R17, R18, R19, R2, R20, R21, R22, R23, R24, R25, R26, R27, R28, R29, R3, R31, R32, R33, R34, R4, R5, R6, R7, R8, R9: (no value), rcl:0207/10
- added U$10, U$11, U$12, U$13, U$14, U$15, U$7, U$8, U$9: RES-7, MIA_LIBRARY-2-2-2:0204/7
- moved S1 194.2 mm to (-38.1, 45.7)
- moved R30 192.6 mm to (-36.8, 64.8)
- moved U$3 192.6 mm to (-24.1, 57.1)
- moved U$5 192.6 mm to (-41.9, 26.7)
- moved U$6 192.6 mm to (-41.9, 19.1)
- moved U$4 192.6 mm to (-24.1, 52.1)
- moved V5 84.2 mm to (101.6, 81.3)
- moved D3 36.8 mm to (71.1, 36.8)
- moved D4 36.8 mm to (86.4, 36.8)
- moved D1 28.5 mm to (71.1, 16.5)
- moved D2 12.0 mm to (86.4, 16.5)
- moved J1 1.27 mm to (5.08, 6.35)
Connections:
- removed net BI/RBO: IC1.4, IC2.5, IC4.4, IC5.5
- removed net N$10: D2.2, R11.2
- removed net N$11: D2.1, R12.2
- removed net N$12: D2.9, R13.1
- removed net N$13: D2.10, R15.1
- removed net N$14: D3.6, R16.2
- removed net N$15: D3.4, R17.2
- removed net N$16: D3.2, R18.2
- removed net N$17: D3.1, R19.2
- removed net N$18: D3.9, R20.1
- removed net N$19: D3.10, R22.1
- removed net N$20: D4.6, R23.2
- removed net N$21: D4.4, R24.2
- removed net N$22: D4.2, R25.2
- removed net N$23: D4.1, R26.2
- removed net N$24: D4.9, R27.1
- removed net N$25: D4.10, R29.1
- removed net N$5: D1.1, R6.2
- removed net N$6: D1.9, R7.1
- removed net N$7: D1.10, R9.1
- removed net N$8: D2.6, R2.2
- removed net N$9: D2.4, R10.2
- new net N$1: D1.8, U$7.1
- net A: no longer D2.7, D3.7, D4.7, IC1.13, R14.2, R21.2, R28.2, R8.1, R8.2
- net A1: now also D2.7; no longer IC2.13, R14.1
- net A2: now also D3.7; no longer IC4.13, R21.1
- net A3: now also D4.7; no longer IC5.13, R28.1
- net B: now also D1.6; no longer IC1.12, R3.1
- net B1: now also D2.6; no longer IC2.12, R2.1
- net B2: now also D3.6; no longer IC4.12, R16.1
- net B3: now also D4.6; no longer IC5.12, R23.1
- net C: now also D1.4; no longer IC1.11, R4.1
- net C1: now also D2.4; no longer IC2.11, R10.1
- net C2: now also D3.4; no longer IC4.11, R17.1
- net C3: now also D4.4; no longer IC5.11, R24.1
- net D: now also D1.2; no longer IC1.10, R5.1
- net D1: now also D2.2; no longer IC2.10, R11.1
- net D2: now also D3.2; no longer IC4.10, R18.1
- net D3: now also D4.2; no longer IC5.10, R25.1
- net DIS: now also U$8.2; no longer R1.1
- net E: now also D1.1; no longer IC1.9, R6.1
- net E1: now also D2.1; no longer IC2.9, R12.1
- net E2: now also D3.1; no longer IC4.9, R19.1
- net E3: now also D4.1; no longer IC5.9, R26.1
- net F: now also D1.9; no longer IC1.15, R7.2
- net F1: now also D2.9; no longer IC2.15, R13.2
- net F2: now also D3.9; no longer IC4.15, R20.2
- net F3: now also D4.9; no longer IC5.15, R27.2
- net G: now also D1.10; no longer IC1.14, R9.2
- net G1: now also D2.10; no longer IC2.14, R15.2
- net G2: now also D3.10; no longer IC4.14, R22.2
- net G3: now also D4.10; no longer IC5.14, R29.2
- net GND: now also U$10.2, U$11.2, U$7.2, U$9.2; no longer D1.3, D1.8, D2.3, D2.8, D3.3, D3.8, D4.3, D4.8, IC1.5, IC1.8, IC2.8, IC4.5, IC4.8, IC5.8
- net N$2: now also D2.8, U$9.1; no longer D1.6, R3.2
- net N$27: now also U$12.2; no longer R32.2
- net N$28: now also U$12.1; no longer R32.1
- net N$29: now also U$13.2; no longer R31.2
- net N$3: now also D3.8, U$10.1; no longer D1.4, R4.2
- net N$30: now also U$13.1; no longer R31.1
- net N$31: now also U$14.2; no longer R34.2
- net N$32: now also U$14.1; no longer R34.1
- net N$33: now also U$15.2; no longer R33.2
- net N$34: now also U$15.1; no longer R33.1
- net N$4: now also D4.8, U$11.1; no longer D1.2, R5.2
- net Q4: no longer IC1.7, IC2.7, IC4.7, IC5.7
- net Q5: no longer IC1.1, IC2.1, IC4.1, IC5.1
- net Q6: no longer IC1.2, IC2.2, IC4.2, IC5.2
- net Q7: no longer IC1.6, IC2.6, IC4.6, IC5.6
- net VCC: now also U$8.1; no longer IC1.16, IC1.3, IC2.16, IC2.3, IC4.16, IC4.3, IC5.16, IC5.3, R1.2
Routing:
- net GND: track 0.00 -> 6.04 mm
Other:
- board size 100 x 80 mm -> 126.7 x 91.4 mm

Commit message: schematics
Parts:
- removed V2: 74107N, 74ttl-din:DIL14
- added IC1, IC2: 74LS48N, 74xx-eu:DIL16
Connections:
- removed net !Q2: V2.6, V3.12
- removed net A2: D3.7
- removed net A3: D4.7
- removed net B2: D3.6
- removed net B3: D4.6
- removed net C2: D3.4
- removed net C3: D4.4
- removed net D2: D3.2
- removed net D3: D4.2
- removed net E2: D3.1
- removed net E3: D4.1
- removed net F2: D3.9
- removed net F3: D4.9
- removed net G2: D3.10
- removed net G3: D4.10
- removed net N$28: U$12.1, V3.8
- removed net N$30: U$13.1, V3.11
- removed net N$32: U$14.1, V3.3
- removed net N$34: U$15.1, V3.6
- removed net TCO\: V2.11
- new net OUT1: U$12.1, U$15.1, V3.3
- new net OUT2: U$13.1, U$14.1, V3.6
- new net Q0: IC1.7, IC7.3
- new net Q3: IC1.6, IC7.7, V5.2
- new net RBI: IC1.4, IC2.5
- net +UB: no longer V2.14
- net -UB: no longer V2.7
- net A: now also D3.7, IC1.13
- net A1: now also D4.7, IC2.13
- net B: now also D3.6, IC1.12
- net B1: now also D4.6, IC2.12
- net C: now also D3.4, IC1.11
- net C1: now also D4.4, IC2.11
- net CLK: no longer V2.9
- net D: now also D3.2, IC1.10
- net D1: now also D4.2, IC2.10
- net E: now also D3.1, IC1.9
- net E1: now also D4.1, IC2.9
- net F: now also D3.9, IC1.15
- net F1: now also D4.9, IC2.15
- net G: now also D3.10, IC1.14
- net G1: now also D4.10, IC2.14
- net GND: now also IC1.5, IC1.8, IC2.8
- net Q1: now also IC1.1, IC7.2
- net Q2: now also IC1.2, IC7.6; no longer V2.5, V3.9
- net Q4: now also IC2.7; no longer IC7.3
- net Q5: now also IC2.1; no longer IC7.2
- net Q6: now also IC2.2; no longer IC7.6
- net Q7: now also IC2.6; no longer IC7.7, V5.2
- net TCO: no longer V2.8
- net VCC: now also IC1.16, IC1.3, IC2.16, IC2.3
- net X: no longer V3.10, V3.13

Commit message: schematics
Parts:
- added S2: (no value), switch:255SB
- moved IC1 222.0 mm to (100.3, 38.1)
- moved U$12 221.4 mm to (22.9, 123.2)
- moved U$13 221.4 mm to (22.9, 118.1)
- moved U$15 216.5 mm to (26.7, 101.6)
- moved IC2 214.2 mm to (77.5, 38.1)
- moved U$14 204.0 mm to (25.4, 94.0)
- moved U$8 135.3 mm to (71.1, 72.4), turned to 90 degrees
- moved IC3 119.4 mm to (80.0, 72.4)
- moved U$9 117.7 mm to (45.7, 49.5), turned to 90 degrees
- moved U$3 111.9 mm to (85.1, 81.3), turned to 270 degrees
- moved R30 111.3 mm to (72.4, 86.4), turned to 180 degrees
- moved U$1 109.6 mm to (31.8, 133.3)
- moved U$5 108.7 mm to (35.6, 102.9)
- moved U$6 108.7 mm to (35.6, 95.2)
- moved U$2 107.8 mm to (15.2, 132.1)
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Connections:
- new net N$5: J1.1, S2.2
- net VCC: now also S2.1; no longer J1.1
Routing:
- net VCC: track 0.00 -> 41.4 mm
- net THR: track 0.00 -> 40.4 mm
- net DIS: track 0.00 -> 31.3 mm
- net CLK: track 0.00 -> 26.6 mm
- net N$5: track 0.00 -> 7.59 mm
- net GND: track 6.04 -> 12.3 mm
- net CV: track 0.00 -> 4.34 mm
Other:
- board size 126.7 x 91.4 mm -> 150.8 x 151.1 mm

Commit message: schematics
Parts:
- moved V5 90.9 mm to (138.4, 21.6)
- moved V1 83.5 mm to (118.1, 20.3)
- moved V4 74.0 mm to (105.4, 94.0)
- moved U$2 62.2 mm to (14.0, 69.8), turned to 180 degrees
- moved U$1 58.6 mm to (14.0, 77.5), turned to 180 degrees
- moved U$5 54.0 mm to (14.0, 53.3), turned to 180 degrees
- moved U$12 53.3 mm to (22.9, 69.8), turned to 180 degrees
- moved S1 51.3 mm to (58.4, 101.6)
- moved U$15 48.4 mm to (22.9, 53.3), turned to 180 degrees
- moved IC1 41.5 mm to (68.6, 11.4)
- moved U$13 40.6 mm to (22.9, 77.5), turned to 180 degrees
- moved U$6 40.5 mm to (14.0, 61.0), turned to 180 degrees
- moved U$4 33.1 mm to (76.2, 97.8)
- moved U$14 33.1 mm to (22.9, 61.0), turned to 180 degrees
- moved IC3 33.1 mm to (77.5, 105.4)
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Routing:
- net TCO0: track 0.00 -> 12.0 mm
- net CLK: track 26.6 -> 37.1 mm

Commit message: sch tweaks
Parts:
- removed IC3: NE555N, linear:DIL08
- removed R30: (no value), pot:3RP/1610N
- removed U$1, U$2, U$5, U$6: LED5MM, MIA-Training:LED5MM
- removed U$10, U$11, U$12, U$13, U$14, U$15, U$7, U$8, U$9: RES-7, MIA_LIBRARY-2-2-2:0204/7
- removed U$3, U$4: (no value), MIA-Training:C025-025X050
- added CLK_PINHD: (no value), MIA-Training:1X03
- added LED1, LED3: RED, MIA_LIBRARY-2-2-2:LED5MM
- added LED2, LED4: GREEN, MIA_LIBRARY-2-2-2:LED5MM
- added R1, R2, R3, R4, R5, R6, R7, R8: 140R, MIA_LIBRARY-2-2-2:0204/7
- moved V5 247.0 mm to (-95.2, 101.6)
- moved V1 235.9 mm to (-96.5, 118.1)
- moved IC6 139.3 mm to (-66.0, 100.3)
- moved S1 139.3 mm to (-78.7, 125.7)
- moved IC2 139.3 mm to (-64.8, 82.5)
- moved IC7 139.3 mm to (-40.6, 100.3)
- moved V4 139.3 mm to (-31.8, 118.1)
- moved IC1 135.6 mm to (-66.0, 27.9)
- moved V3 135.6 mm to (-39.4, 36.8)
- moved D1 101.2 mm to (123.2, 74.9)
- moved D2 98.9 mm to (135.9, 74.9)
- moved D3 91.6 mm to (121.9, 19.1)
- moved D4 89.0 mm to (134.6, 19.1)
Connections:
- removed net CV: IC3.5, U$3.2
- removed net DIS: IC3.7, R30.2, U$8.2
- removed net THR: IC3.2, IC3.6, R30.3, U$4.1
- net CLK: now also CLK_PINHD.3; no longer IC3.3
- net GND: now also CLK_PINHD.2, LED1.K, LED2.K, LED3.K, LED4.K, R5.2, R6.2, R7.2, R8.2; no longer IC3.1, U$1.K, U$10.2, U$11.2, U$2.K, U$3.1, U$4.2, U$5.K, U$6.K, U$7.2, U$9.2
- net N$1: now also R5.1; no longer U$7.1
- net N$2: now also R7.1; no longer U$9.1
- net N$27: now also LED1.A, R1.2; no longer U$12.2, U$2.A
- net N$29: now also LED2.A, R2.2; no longer U$1.A, U$13.2
- net N$3: now also R6.1; no longer U$10.1
- net N$31: now also LED3.A, R4.2; no longer U$14.2, U$6.A
- net N$33: now also LED4.A, R3.2; no longer U$15.2, U$5.A
- net N$4: now also R8.1; no longer U$11.1
- net OUT1: now also R1.1, R3.1; no longer U$12.1, U$15.1
- net OUT2: now also R2.1, R4.1; no longer U$13.1, U$14.1
- net VCC: now also CLK_PINHD.1; no longer IC3.4, IC3.8, R30.1, U$8.1
Routing:
- net VCC: track 41.4 -> 0.00 mm
- net THR: track 40.4 -> 0.00 mm
- net DIS: track 31.3 -> 0.00 mm
- net GND: track 12.3 -> 6.04 mm
- net CV: track 4.34 -> 0.00 mm

Commit message: sch tweaks
Parts:
- moved LED1 183.4 mm to (53.3, 80.0)
- moved LED2 183.4 mm to (53.3, 72.4)
- moved R7 177.6 mm to (85.1, 92.7)
- moved LED3 169.8 mm to (53.3, 26.7)
- moved IC6 167.1 mm to (91.4, 44.5)
- moved LED4 164.7 mm to (53.3, 19.1)
- moved V4 164.7 mm to (115.6, 44.5)
- moved R8 163.4 mm to (85.1, 7.62), turned to 270 degrees
- moved IC2 157.7 mm to (91.4, 61.0)
- moved S1 137.7 mm to (40.6, 57.1), turned to 180 degrees
- moved IC1 136.1 mm to (66.0, 61.0)
- moved V1 128.9 mm to (19.1, 61.0)
- moved V5 127.8 mm to (19.1, 44.5)
- moved R6 126.2 mm to (72.4, 7.62), turned to 270 degrees
- moved IC7 120.4 mm to (66.0, 44.5)
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Connections:
- removed net +UB: V1.14, V3.14, V4.14, V5.14
- removed net -UB: V1.7, V3.7, V4.7, V5.7
- net GND: now also V1.7, V3.7, V4.7, V5.7
- net N$3: now also D3.3; no longer D3.8
- net N$4: now also D4.3; no longer D4.8
- net VCC: now also V1.14, V3.14, V4.14, V5.14
Routing:
- net GND: track 6.04 -> 219.6 mm
- net CLK: track 37.0 -> 123.6 mm
- net TCO0: track 12.0 -> 0.00 mm
- net VCC: track 0.00 -> 10.2 mm
- net N$33: track 0.00 -> 3.81 mm
- net N$31: track 0.00 -> 3.81 mm
- net N$29: track 0.00 -> 3.81 mm
- net N$27: track 0.00 -> 3.81 mm
- net N$2: track 0.00 -> 3.81 mm
- net N$1: track 0.00 -> 3.81 mm
- net N$4: track 0.00 -> 3.81 mm
- net N$3: track 0.00 -> 3.81 mm
Other:
- board size 150.8 x 151.1 mm -> 150.8 x 111.8 mm

Commit message: board
Parts:
- moved R5 83.9 mm to (76.2, 8.89), turned to 270 degrees
- moved R7 83.9 mm to (88.9, 8.89), turned to 270 degrees
- moved LED3 68.3 mm to (41.9, 94.0)
- moved R3 68.3 mm to (33.0, 86.4)
- moved R4 68.3 mm to (33.0, 94.0)
- moved LED4 68.1 mm to (43.2, 86.4), turned to 180 degrees
- moved S1 66.6 mm to (74.9, 114.3)
- moved V5 60.3 mm to (71.1, 74.9)
- moved D1 53.5 mm to (76.2, 24.1)
- moved D2 53.5 mm to (88.9, 24.1)
- moved IC2 51.3 mm to (57.1, 22.9)
- moved IC1 50.3 mm to (57.1, 11.4)
- moved LED1 43.0 mm to (12.7, 94.0), turned to 180 degrees
- moved LED2 43.0 mm to (12.7, 86.4), turned to 180 degrees
- moved D3 30.5 mm to (102.9, 24.1)
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Connections:
- net !Q1 renamed !OQ1
- new net OQ1: V1.5, V3.1
- net GND: now also D1.3, D2.3, D3.8, D4.8
- net LD: now also V5.2; no longer V5.1
- net Q1: no longer V1.5, V3.1
- net Q3: now also V5.1; no longer V5.2
Routing:
- net GND: track 219.6 -> 7.06 mm
- net CLK: track 123.6 -> 0.80 mm
- net VCC: track 10.2 -> 0.00 mm
- net N$33: track 3.81 -> 0.00 mm
- net N$31: track 3.81 -> 0.00 mm
- net N$29: track 3.81 -> 0.00 mm
- net N$27: track 3.81 -> 0.00 mm
- net N$2: track 3.81 -> 0.00 mm
- net N$1: track 3.81 -> 0.00 mm
- net N$4: track 3.81 -> 0.00 mm
- net N$3: track 3.81 -> 0.00 mm
Other:
- board size 150.8 x 111.8 mm -> 129.2 x 101.6 mm

Commit message: backup
Parts:
- removed S2: (no value), switch:255SB
- added V2: 74107N, 74ttl-din:DIL14
- moved CLK_PINHD 107.9 mm to (112.5, 7.69), turned to 180 degrees
- moved S1 90.1 mm to (143.5, 55.9), turned to 270 degrees
- moved D1 85.3 mm to (15.2, 83.8)
- moved R5 85.3 mm to (15.2, 68.6)
- moved D2 85.3 mm to (27.9, 83.8)
- moved R7 85.3 mm to (27.9, 68.6)
- moved V1 75.0 mm to (64.8, 15.2)
- moved V5 69.5 mm to (35.6, 15.2)
- moved LED4 68.8 mm to (111.8, 81.3)
- moved LED3 68.8 mm to (110.5, 88.9)
- moved R3 68.8 mm to (101.6, 81.3)
- moved R4 68.8 mm to (101.6, 88.9)
- moved D4 63.5 mm to (137.2, 83.8)
- moved R8 63.5 mm to (137.2, 68.6)
- moved D3 63.5 mm to (124.5, 83.8)
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Connections:
- removed net N$5: J1.1, S2.2
- new net +UB: V2.14
- new net -UB: V2.7
- net !OQ1: now also V2.2; no longer V1.6
- net CLK: now also V2.12; no longer V1.9
- net GND: now also D1.8, D2.8; no longer D1.3, D2.3
- net LD: now also V5.8; no longer V5.2
- net N$1: now also D1.3; no longer D1.8
- net N$2: now also D2.3; no longer D2.8
- net OQ1: now also V2.3; no longer V1.5
- net Q3: now also V5.9; no longer V5.1
- net TCO: now also V2.1, V2.4, V4.11; no longer V1.11, V1.8, V4.3
- net TCO0: now also V4.12; no longer V4.1
- net TCO1: now also V4.13; no longer V4.2
- net VCC: now also J1.1; no longer S2.1
Routing:
- net TCO: track 0.00 -> 114.7 mm, vias 0 -> 2
- net CLK: track 0.80 -> 108.6 mm
- net Q: track 0.00 -> 51.2 mm, vias 0 -> 2
- net GND: track 7.06 -> 44.3 mm
- net VCC: track 0.00 -> 27.5 mm
- net N$5: track 7.59 -> 0.00 mm
- net Q7: track 0.00 -> 4.34 mm
- net Q5: track 0.00 -> 1.27 mm
Other:
- board size 129.2 x 101.6 mm -> 149.5 x 99 mm
