File: traffic_light.sch (EAGLE design)
At the start: 58 parts, among them IC1 74LS48N, IC2 74LS48N, IC3 NE555N, IC4 74LS48N, IC5 74LS48N, IC6 74190N, IC7 74190N

Commit message: commit
Parts:
- removed IC1, IC2, IC4, IC5: 74LS48N, 74xx-eu:74LS48N
- removed R1, R10, R11, R12, R13, R14, R15, R16, R17, R18, R19, R2, R20, R21, R22, R23, R24, R25, R26, R27, R28, R29, R3, R31, R32, R33, R34, R4, R5, R6, R7, R8, R9: (no value), rcl:R-EU_0207/10
- added U$10, U$11, U$12, U$13, U$14, U$15, U$7, U$8, U$9: RES-7, MIA_LIBRARY-2-2-2:RES-7
Connections:
- removed net BI/RBO: IC1A.BI/RBO, IC2A.RBI, IC4A.BI/RBO, IC5A.RBI
- removed net N$10: D2.D, R11.2
- removed net N$11: D2.E, R12.2
- removed net N$12: D2.F, R13.1
- removed net N$13: D2.G, R15.1
- removed net N$14: D3.B, R16.2
- removed net N$15: D3.C, R17.2
- removed net N$16: D3.D, R18.2
- removed net N$17: D3.E, R19.2
- removed net N$18: D3.F, R20.1
- removed net N$19: D3.G, R22.1
- removed net N$20: D4.B, R23.2
- removed net N$21: D4.C, R24.2
- removed net N$22: D4.D, R25.2
- removed net N$23: D4.E, R26.2
- removed net N$24: D4.F, R27.1
- removed net N$25: D4.G, R29.1
- removed net N$5: D1.E, R6.2
- removed net N$6: D1.F, R7.1
- removed net N$7: D1.G, R9.1
- removed net N$8: D2.B, R2.2
- removed net N$9: D2.C, R10.2
- new net N$1: D1.CK2, U$7.1
- net A: no longer D2.A, D3.A, D4.A, IC1A.A, R14.2, R21.2, R28.2, R8.1, R8.2
- net A1: now also D2.A; no longer IC2A.A, R14.1
- net A2: now also D3.A; no longer IC4A.A, R21.1
- net A3: now also D4.A; no longer IC5A.A, R28.1
- net B: now also D1.B; no longer IC1A.B, R3.1
- net B1: now also D2.B; no longer IC2A.B, R2.1
- net B2: now also D3.B; no longer IC4A.B, R16.1
- net B3: now also D4.B; no longer IC5A.B, R23.1
- net C: now also D1.C; no longer IC1A.C, R4.1
- net C1: now also D2.C; no longer IC2A.C, R10.1
- net C2: now also D3.C; no longer IC4A.C, R17.1
- net C3: now also D4.C; no longer IC5A.C, R24.1
- net D: now also D1.D; no longer IC1A.D, R5.1
- net D1: now also D2.D; no longer IC2A.D, R11.1
- net D2: now also D3.D; no longer IC4A.D, R18.1
- net D3: now also D4.D; no longer IC5A.D, R25.1
- net DIS: now also U$8.2; no longer R1.1
- net E: now also D1.E; no longer IC1A.E, R6.1
- net E1: now also D2.E; no longer IC2A.E, R12.1
- net E2: now also D3.E; no longer IC4A.E, R19.1
- net E3: now also D4.E; no longer IC5A.E, R26.1
- net F: now also D1.F; no longer IC1A.F, R7.2
- net F1: now also D2.F; no longer IC2A.F, R13.2
- net F2: now also D3.F; no longer IC4A.F, R20.2
- net F3: now also D4.F; no longer IC5A.F, R27.2
- net G: now also D1.G; no longer IC1A.G, R9.2
- net G1: now also D2.G; no longer IC2A.G, R15.2
- net G2: now also D3.G; no longer IC4A.G, R22.2
- net G3: now also D4.G; no longer IC5A.G, R29.2
- net GND: now also U$10.2, U$11.2, U$7.2, U$9.2; no longer D1.CK1, D1.CK2, D2.CK1, D2.CK2, D3.CK1, D3.CK2, D4.CK1, D4.CK2, IC1A.RBI, IC4A.RBI
- net N$2: now also D2.CK2, U$9.1; no longer D1.B, R3.2
- net N$27: now also U$12.2; no longer R32.2
- net N$28: now also U$12.1; no longer R32.1
- net N$29: now also U$13.2; no longer R31.2
- net N$3: now also D3.CK2, U$10.1; no longer D1.C, R4.2
- net N$30: now also U$13.1; no longer R31.1
- net N$31: now also U$14.2; no longer R34.2
- net N$32: now also U$14.1; no longer R34.1
- net N$33: now also U$15.2; no longer R33.2
- net N$34: now also U$15.1; no longer R33.1
- net N$4: now also D4.CK2, U$11.1; no longer D1.D, R5.2
- net Q4: no longer IC1A.IA, IC2A.IA, IC4A.IA, IC5A.IA
- net Q5: no longer IC1A.IB, IC2A.IB, IC4A.IB, IC5A.IB
- net Q6: no longer IC1A.IC, IC2A.IC, IC4A.IC, IC5A.IC
- net Q7: no longer IC1A.ID, IC2A.ID, IC4A.ID, IC5A.ID
- net VCC: now also U$8.1; no longer IC1A.LT, IC2A.LT, IC4A.LT, IC5A.LT, R1.2
Other:
- moved on the sheet: D1, D2, D3, D4, IC3, IC6, IC7, J1, R30, S1, U$1, U$2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

Commit message: schematics
Parts:
- removed V2: 74107N, 74ttl-din:74107N
- added IC1, IC2: 74LS48N, 74xx-eu:74LS48N
Connections:
- removed net !Q2: V2/2.!Q, V3/4.A
- removed net A2: D3.A
- removed net A3: D4.A
- removed net B2: D3.B
- removed net B3: D4.B
- removed net C2: D3.C
- removed net C3: D4.C
- removed net D2: D3.D
- removed net D3: D4.D
- removed net E2: D3.E
- removed net E3: D4.E
- removed net F2: D3.F
- removed net F3: D4.F
- removed net G2: D3.G
- removed net G3: D4.G
- removed net N$28: U$12.1, V3/3.Y
- removed net N$30: U$13.1, V3/4.Y
- removed net N$32: U$14.1, V3/1.Y
- removed net N$34: U$15.1, V3/2.Y
- removed net TCO\: V2/2.K
- new net OUT1: U$12.1, U$15.1, V3/1.Y
- new net OUT2: U$13.1, U$14.1, V3/2.Y
- new net Q0: IC1A.IA, IC7A.QA
- new net Q3: IC1A.ID, IC7A.QD, V5/1.Y
- new net RBI: IC1A.BI/RBO, IC2A.RBI
- net A: now also D3.A, IC1A.A
- net A1: now also D4.A, IC2A.A
- net B: now also D3.B, IC1A.B
- net B1: now also D4.B, IC2A.B
- net C: now also D3.C, IC1A.C
- net C1: now also D4.C, IC2A.C
- net CLK: no longer V2/2.CLK
- net D: now also D3.D, IC1A.D
- net D1: now also D4.D, IC2A.D
- net E: now also D3.E, IC1A.E
- net E1: now also D4.E, IC2A.E
- net F: now also D3.F, IC1A.F
- net F1: now also D4.F, IC2A.F
- net G: now also D3.G, IC1A.G
- net G1: now also D4.G, IC2A.G
- net GND: now also IC1A.RBI
- net Q1: now also IC1A.IB, IC7A.QB
- net Q2: now also IC1A.IC, IC7A.QC; no longer V2/2.Q, V3/3.A
- net Q4: now also IC2A.IA; no longer IC7A.QA
- net Q5: now also IC2A.IB; no longer IC7A.QB
- net Q6: now also IC2A.IC; no longer IC7A.QC
- net Q7: now also IC2A.ID; no longer IC7A.QD, V5/1.Y
- net TCO: no longer V2/2.J
- net VCC: now also IC1A.LT, IC2A.LT
- net X: no longer V3/3.B, V3/4.B
Other:
- moved on the sheet: S1, U$1, U$12, U$13, U$14, U$15, U$2, U$5, U$6, V3/1, V3/2

Commit message: schematics
Parts:
- added S2: (no value), switch:255SB
Connections:
- new net N$5: J1.1, S2.P
- net VCC: now also S2.O; no longer J1.1
Other:
- moved on the sheet: D1, D2, D3, D4, IC1, IC2, IC3, J1, R30, S1, U$1, U$10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

Commit message: sch tweaks
Parts:
- removed IC3: NE555N, linear:NE555N
- removed R30: (no value), pot:3RP/1610N
- removed U$1, U$2, U$5, U$6: LED5MM, MIA-Training:LED5MM
- removed U$10, U$11, U$12, U$13, U$14, U$7, U$8, U$9: RES-7, MIA_LIBRARY-2-2-2:RES-7
- removed U$3, U$4: (no value), MIA-Training:CAPACITOR
- added CLK_PINHD: (no value), MIA-Training:PINHD-1X3
- added LED1, LED3: RED, MIA_LIBRARY-2-2-2:LED5MM
- added LED2, LED4: GREEN, MIA_LIBRARY-2-2-2:LED5MM
- added R1, R2, R3, R5, R6, R7, R8: 140R, MIA_LIBRARY-2-2-2:RES-7
- R4: value RES-7 -> 140R
- renumbered U$15 to R4
Connections:
- removed net CV: IC3.CV, U$3.2
- removed net DIS: IC3.DIS, R30.S, U$8.2
- removed net THR: IC3.THR, IC3.TR, R30.E, U$4.1
- net CLK: now also CLK_PINHD.3; no longer IC3.Q
- net GND: now also CLK_PINHD.2, LED1.C, LED2.C, LED3.C, LED4.C, R5.2, R6.2, R7.2, R8.2; no longer IC3.GND, U$1.C, U$10.2, U$11.2, U$2.C, U$3.1, U$4.2, U$5.C, U$6.C, U$7.2, U$9.2
- net N$1: now also R5.1; no longer U$7.1
- net N$2: now also R7.1; no longer U$9.1
- net N$27: now also LED1.A, R1.2; no longer U$12.2, U$2.A
- net N$29: now also LED2.A, R2.2; no longer U$1.A, U$13.2
- net N$3: now also R6.1; no longer U$10.1
- net N$31: now also LED3.A, R4.2; no longer U$14.2, U$6.A
- net N$33: now also LED4.A, R3.2; no longer R4.2, U$5.A
- net N$4: now also R8.1; no longer U$11.1
- net OUT1: now also R1.1, R3.1; no longer R4.1, U$12.1
- net OUT2: now also R2.1, R4.1; no longer U$13.1, U$14.1
- net VCC: now also CLK_PINHD.1; no longer IC3.R, IC3.V+, R30.A, U$8.1
Other:
- moved on the sheet: D1, D2, D3, D4, J1, S2

Commit message: sch tweaks
Connections:
- net GND: now also V1/-UB.-UB, V3/-UB.-UB, V4/-UB.-UB, V5/-UB.-UB
- net N$3: now also D3.CK1; no longer D3.CK2
- net N$4: now also D4.CK1; no longer D4.CK2
- net VCC: now also V1/+UB.+UB, V3/+UB.+UB, V4/+UB.+UB, V5/+UB.+UB
Other:
- moved on the sheet: CLK_PINHD, R6, R8
Changed lines of the file:
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@@
 <attribute name="VALUE" x="162.56" y="68.58" size="1.778" layer="96"/>
 </instance>
-<instance part="R6" gate="G$1" x="182.88" y="73.66" smashed="yes" grouprefs="DISPLAY">
-<attribute name="NAME" x="179.07" y="75.1586" size="1.778" layer="95"/>
-<attribute name="VALUE" x="179.07" y="70.358" size="1.778" layer="96"/>
+<instance part="R6" gate="G$1" x="182.88" y="76.2" smashed="yes" grouprefs="DISPLAY">
+<attribute name="NAME" x="179.07" y="77.6986" size="1.778" layer="95"/>
+<attribute name="VALUE" x="179.07" y="72.898" size="1.778" layer="96"/>
 </instance>
 <instance part="D4" gate="G$1" x="213.36" y="78.74" smashed="yes" grouprefs="DISPLAY">
@@
 <attribute name="VALUE" x="208.28" y="68.58" size="1.778" layer="96"/>
 </instance>
-<instance part="R8" gate="G$1" x="228.6" y="73.66" smashed="yes" grouprefs="DISPLAY">
-<attribute name="NAME" x="224.79" y="75.1586" size="1.778" layer="95"/>
-<attribute name="VALUE" x="224.79" y="70.358" size="1.778" layer="96"/>
+<instance part="R8" gate="G$1" x="228.6" y="76.2" smashed="yes" grouprefs="DISPLAY">
+<attribute name="NAME" x="224.79" y="77.6986" size="1.778" layer="95"/>
+<attribute name="VALUE" x="224.79" y="72.898" size="1.778" layer="96"/>
 </instance>
 <instance part="R1" gate="G$1" x="210.82" y="167.64" smashed="yes" grouprefs="LEDS">
@@
 <attribute name="VALUE" x="274.955" y="80.01" size="1.778" layer="96"/>
 </instance>
-<instance part="CLK_PINHD" gate="A" x="78.74" y="106.68" smashed="yes" grouprefs="CLOCK">
-<attribute name="NAME" x="72.39" y="112.395" size="1.778" layer="95"/>
-<attribute name="VALUE" x="72.39" y="99.06" size="1.778" layer="96"/>
+<instance part="CLK_PINHD" gate="A" x="83.82" y="109.22" smashed="yes" grouprefs="CLOCK">
+<attribute name="NAME" x="77.47" y="114.935" size="1.778" layer="95"/>
+<attribute name="VALUE" x="77.47" y="101.6" size="1.778" layer="96"/>
 </instance>
 <instance part="LED1" gate="G$1" x="220.98" y="167.64" smashed="yes" rot="R90">
@@
 <attribute name="NAME" x="225.552" y="143.256" size="1.778" layer="95" rot="R180"/>
 <attribute name="VALUE" x="225.552" y="145.415" size="1.778" layer="96" rot="R180"/>
+</instance>
+<instance part="V5" gate="/+UB" x="116.84" y="167.64" smashed="yes" rot="R90" grouprefs="COUNTER">
+<attribute name="NAME" x="118.11" y="168.91" size="1.524" layer="95" rot="R90"/>
+</instance>
+<instance part="V5" gate="/-UB" x="132.08" y="167.64" smashed="yes" rot="R90" grouprefs="COUNTER">
+<attribute name="NAME" x="132.08" y="168.91" size="1.524" layer="95" rot="R90"/>
+</instance>
+<instance part="V4" gate="/+UB" x="81.28" y="162.56" smashed="yes" rot="R270" grouprefs="COUNTER_CONTROLLER">
+<attribute name="NAME" x="80.01" y="161.29" size="1.524" layer="95" rot="R270"/>
+</instance>
+<instance part="V4" gate="/-UB" x="81.28" y="167.64" smashed="yes" rot="R90" grouprefs="COUNTER_CONTROLLER">
+<attribute name="NAME" x="81.28" y="168.91" size="1.524" layer="95" rot="R90"/>
+</instance>
+<instance part="V1" gate="/+UB" x="60.96" y="129.54" smashed="yes" rot="R90" grouprefs="COUNTER_CONTROLLER">
+<attribute name="NAME" x="62.23" y="130.81" size="1.524" layer="95" rot="R90"/>
+</instance>
+<instance part="V1" gate="/-UB" x="93.98" y="129.54" smashed="yes" rot="R180" grouprefs="COUNTER_CONTROLLER">
+<attribute name="NAME" x="92.71" y="129.54" size="1.524" layer="95" rot="R180"/>
+</instance>
+<instance part="V3" gate="/+UB" x="185.42" y="160.02" smashed="yes" rot="R270">
+<attribute name="NAME" x="184.15" y="158.75" size="1.524" layer="95" rot="R270"/>
+</instance>
+<instance part="V3" gate="/-UB" x="185.42" y="162.56" smashed="yes" rot="R90">
+<attribute name="NAME" x="185.42" y="163.83" size="1.524" layer="95" rot="R90"/>
 </instance>
 </instances>
@@
 <segment>
 <pinref part="CLK_PINHD" gate="A" pin="1"/>
-<wire x1="76.2" y1="109.22" x2="71.12" y2="109.22" width="0.1524" layer="91" grouprefs="CLOCK"/>
-<label x="71.12" y="109.22" size="1.27" layer="95" rot="R180" xref="yes" grouprefs="CLOCK"/>
+<wire x1="81.28" y1="111.76" x2="76.2" y2="111.76" width="0.1524" layer="91" grouprefs="CLOCK"/>
+<label x="76.2" y="111.76" size="1.27" layer="95" rot="R180" xref="yes" grouprefs="CLOCK"/>
+</segment>
+<segment>
+<pinref part="V5" gate="/+UB" pin="+UB"/>
+<wire x1="114.3" y1="167.64" x2="111.76" y2="167.64" width="0.1524" layer="91" grouprefs="COUNTER"/>
+<label x="111.76" y="167.64" size="1.27" layer="95" rot="R180" xref="yes" grouprefs="COUNTER"/>
+</segment>
+<segment>
+<pinref part="V4" gate="/+UB" pin="+UB"/>
+<wire x1="83.82" y1="162.56" x2="86.36" y2="162.56" width="0.1524" layer="91" grouprefs="COUNTER_CONTROLLER"/>
+<label x="86.36" y="162.56" size="1.27" layer="95" xref="yes" grouprefs="COUNTER_CONTROLLER"/>
+</segment>
+<segment>
+<pinref part="V1" gate="/+UB" pin="+UB"/>
+<wire x1="58.42" y1="129.54" x2="55.88" y2="129.54" width="0.1524" layer="91" grouprefs="COUNTER_CONTROLLER"/>
+<label x="55.88" y="129.54" size="1.27" layer="95" rot="R180" xref="yes" grouprefs="COUNTER_CONTROLLER"/>
+</segment>
+<segment>
+<pinref part="V3" gate="/+UB" pin="+UB"/>
+<wire x1="187.96" y1="160.02" x2="190.5" y2="160.02" width="0.1524" layer="91"/>
+<label x="190.5" y="160.02" size="1.27" layer="95" xref="yes"/>
 </segment>
 </net>
@@
 <segment>
 <pinref part="R6" gate="G$1" pin="2"/>
-<wire x1="187.96" y1="73.66" x2="190.5" y2="73.66" width="0.1524" layer="91" grouprefs="DISPLAY"/>
-<label x="190.5" y="73.66" size="1.27" layer="95" xref="yes" grouprefs="DISPLAY"/>
+<wire x1="187.96" y1="76.2" x2="190.5" y2="76.2" width="0.1524" layer="91" grouprefs="DISPLAY"/>
+<label x="190.5" y="76.2" size="1.27" layer="95" xref="yes" grouprefs="DISPLAY"/>
 </segment>
 <segment>
 <pinref part="R8" gate="G$1" pin="2"/>
-<wire x1="233.68" y1="73.66" x2="236.22" y2="73.66" width="0.1524" layer="91" grouprefs="DISPLAY"/>
-<label x="236.22" y="73.66" size="1.27" layer="95" xref="yes" grouprefs="DISPLAY"/>
+<wire x1="233.68" y1="76.2" x2="236.22" y2="76.2" width="0.1524" layer="91" grouprefs="DISPLAY"/>
+<label x="236.22" y="76.2" size="1.27" layer="95" xref="yes" grouprefs="DISPLAY"/>
 </segment>
 <segment>
@@
 <segment>
 <pinref part="CLK_PINHD" gate="A" pin="2"/>
-<wire x1="76.2" y1="106.68" x2="71.12" y2="106.68" width="0.1524" layer="91" grouprefs="CLOCK"/>
-<label x="71.12" y="106.68" size="1.27" layer="95" rot="R180" xref="yes" grouprefs="CLOCK"/>
+<wire x1="81.28" y1="109.22" x2="76.2" y2="109.22" width="0.1524" layer="91" grouprefs="CLOCK"/>
+<label x="76.2" y="109.22" size="1.27" layer="95" rot="R180" xref="yes" grouprefs="CLOCK"/>
+</segment>
+<segment>
+<pinref part="V5" gate="/-UB" pin="-UB"/>
+<wire x1="134.62" y1="167.64" x2="137.16" y2="167.64" width="0.1524" layer="91" grouprefs="COUNTER"/>
+<label x="137.16" y="167.64" size="1.27" layer="95" xref="yes" grouprefs="COUNTER"/>
+</segment>
+<segment>
+<pinref part="V4" gate="/-UB" pin="-UB"/>
+<wire x1="83.82" y1="167.64" x2="86.36" y2="167.64" width="0.1524" layer="91" grouprefs="COUNTER_CONTROLLER"/>
+<label x="86.36" y="167.64" size="1.27" layer="95" xref="yes" grouprefs="COUNTER_CONTROLLER"/>
+</segment>
+<segment>
+<pinref part="V1" gate="/-UB" pin="-UB"/>
+<wire x1="93.98" y1="132.08" x2="93.98" y2="134.62" width="0.1524" layer="91" grouprefs="COUNTER_CONTROLLER"/>
+<label x="93.98" y="134.62" size="1.27" layer="95" rot="R90" xref="yes" grouprefs="COUNTER_CONTROLLER"/>
+</segment>
+<segment>
+<pinref part="V3" gate="/-UB" pin="-UB"/>
+<wire x1="187.96" y1="162.56" x2="190.5" y2="162.56" width="0.1524" layer="91"/>
+<label x="190.5" y="162.56" size="1.27" layer="95" xref="yes"/>
 </segment>
 </net>
@@
 <segment>
 <pinref part="CLK_PINHD" gate="A" pin="3"/>
-<wire x1="76.2" y1="104.14" x2="71.12" y2="104.14" width="0.1524" layer="91" grouprefs="CLOCK"/>
-<label x="71.12" y="104.14" size="1.27" layer="95" rot="R180" xref="yes" grouprefs="CLOCK"/>
+<wire x1="81.28" y1="106.68" x2="76.2" y2="106.68" width="0.1524" layer="91" grouprefs="CLOCK"/>
+<label x="76.2" y="106.68" size="1.27" layer="95" rot="R180" xref="yes" grouprefs="CLOCK"/>
 </segment>
 </net>
@@
 </segment>
 </net>
-<net name="N$3" class="0">
-<segment>
-<pinref part="D3" gate="G$1" pin="CK2"/>
-<pinref part="R6" gate="G$1" pin="1"/>
-<wire x1="175.26" y1="73.66" x2="177.8" y2="73.66" width="0.1524" layer="91" grouprefs="DISPLAY"/>
-</segment>
-</net>
-<net name="N$4" class="0">
-<segment>
-<pinref part="D4" gate="G$1" pin="CK2"/>
-<pinref part="R8" gate="G$1" pin="1"/>
-<wire x1="220.98" y1="73.66" x2="223.52" y2="73.66" width="0.1524" layer="91" grouprefs="DISPLAY"/>
-</segment>
-</net>
 <net name="RBI" class="0">
 <segment>
@@
 </segment>
 </net>
+<net name="N$3" class="0">
+<segment>
+<pinref part="D3" gate="G$1" pin="CK1"/>
+<pinref part="R6" gate="G$1" pin="1"/>
+<wire x1="175.26" y1="76.2" x2="177.8" y2="76.2" width="0.1524" layer="91"/>
+</segment>
+</net>
+<net name="N$4" class="0">
+<segment>
+<pinref part="D4" gate="G$1" pin="CK1"/>
+<pinref part="R8" gate="G$1" pin="1"/>
+<wire x1="220.98" y1="76.2" x2="223.52" y2="76.2" width="0.1524" layer="91"/>
+</segment>
+</net>

Commit message: board
Connections:
- net !Q1 renamed !OQ1
- new net OQ1: V1/2.Q, V3/1.A
- net GND: now also D1.CK1, D2.CK1, D3.CK2, D4.CK2
- net LD: now also V5/1.Y; no longer V5/1.A
- net Q1: no longer V1/2.Q, V3/1.A
- net Q3: now also V5/1.A; no longer V5/1.Y

Commit message: backup
Parts:
- removed S2: (no value), switch:255SB
- added V2: 74107N, 74ttl-din:74107N
Connections:
- removed net N$5: J1.1, S2.P
- net !OQ1: now also V2/1.!Q; no longer V1/2.!Q
- net CLK: now also V2/1.CLK; no longer V1/2.CLK
- net GND: now also D1.CK2, D2.CK2; no longer D1.CK1, D2.CK1
- net LD: now also V5/4.Y; no longer V5/1.Y
- net N$1: now also D1.CK1; no longer D1.CK2
- net N$2: now also D2.CK1; no longer D2.CK2
- net OQ1: now also V2/1.Q; no longer V1/2.Q
- net Q3: now also V5/4.A; no longer V5/1.A
- net TCO: now also V2/1.J, V2/1.K, V4/4.Y; no longer V1/2.J, V1/2.K, V4/1.Y
- net TCO0: now also V4/4.A; no longer V4/1.A
- net TCO1: now also V4/4.B; no longer V4/1.B
- net VCC: now also J1.1; no longer S2.O
Other:
- moved on the sheet: R5, R7
